Commit message: broken one

File: security_robot/src/sr_bringup/descriptions/security_robot.urdf.xacro (robot description, xacro)
@@ -1,5 +1,6 @@
 <?xml version="1.0" ?>
 <robot xmlns:xacro="http://www.ros.org/wiki/xacro" name="security_robot">
-  <xacro:include filename="$(find sec_rob_pkg)/descriptions/materials.xacro" />
+  <xacro:property name="pkg_name" value="sr_bringup" />
+  <xacro:include filename="$(find ${pkg_name})/descriptions/materials.xacro" />
   <link name="base_link"/>
   <link name="chassis">
@@ -7,5 +8,5 @@
       <origin xyz="0 0 0" rpy="0 0 0"/>
       <geometry>
-        <mesh filename="file://$(find sec_rob_pkg)/meshes/chassis.dae"/>
+        <mesh filename="file://$(find ${pkg_name})/meshes/chassis.dae"/>
       </geometry>
       <material name="orange"/>
@@ -14,5 +15,5 @@
       <origin xyz="0 0 0" rpy="0 0 0"/>
       <geometry>
-        <mesh filename="file://$(find sec_rob_pkg)/meshes/chassis.dae"/>
+        <mesh filename="file://$(find ${pkg_name})/meshes/chassis.dae"/>
       </geometry>
     </collision>
@@ -27,5 +28,5 @@
       <origin xyz="0 0 0" rpy="0 0 0"/>
       <geometry>
-        <mesh filename="file://$(find sec_rob_pkg)/meshes/holder.dae"/>
+        <mesh filename="file://$(find ${pkg_name})/meshes/holder.dae"/>
       </geometry>
       <material name="black"/>
@@ -34,5 +35,5 @@
       <origin xyz="0 0 0" rpy="0 0 0"/>
       <geometry>
-        <mesh filename="file://$(find sec_rob_pkg)/meshes/holder.dae"/>
+        <mesh filename="file://$(find ${pkg_name})/meshes/holder.dae"/>
       </geometry>
     </collision>
@@ -47,5 +48,5 @@
       <origin xyz="0 0 0" rpy="0 0 0"/>
       <geometry>
-        <mesh filename="file://$(find sec_rob_pkg)/meshes/holder.dae"/>
+        <mesh filename="file://$(find ${pkg_name})/meshes/holder.dae"/>
       </geometry>
       <material name="black"/>
@@ -54,5 +55,5 @@
       <origin xyz="0 0 0" rpy="0 0 0"/>
       <geometry>
-        <mesh filename="file://$(find sec_rob_pkg)/meshes/holder.dae"/>
+        <mesh filename="file://$(find ${pkg_name})/meshes/holder.dae"/>
       </geometry>
     </collision>
@@ -67,5 +68,5 @@
       <origin xyz="0 0 0" rpy="0 0 0"/>
       <geometry>
-        <mesh filename="file://$(find sec_rob_pkg)/meshes/wheel.dae"/>
+        <mesh filename="file://$(find ${pkg_name})/meshes/wheel.dae"/>
       </geometry>
       <material name="black"/>
@@ -74,5 +75,5 @@
       <origin xyz="0 0 0" rpy="0 0 0"/>
       <geometry>
-        <mesh filename="file://$(find sec_rob_pkg)/meshes/wheel.dae"/>
+        <mesh filename="file://$(find ${pkg_name})/meshes/wheel.dae"/>
       </geometry>
     </collision>
@@ -87,5 +88,5 @@
       <origin xyz="0 0 0" rpy="0 0 0"/>
       <geometry>
-        <mesh filename="file://$(find sec_rob_pkg)/meshes/wheel.dae"/>
+        <mesh filename="file://$(find ${pkg_name})/meshes/wheel.dae"/>
       </geometry>
       <material name="black"/>
@@ -94,5 +95,5 @@
       <origin xyz="0 0 0" rpy="0 0 0"/>
       <geometry>
-        <mesh filename="file://$(find sec_rob_pkg)/meshes/wheel.dae"/>
+        <mesh filename="file://$(find ${pkg_name})/meshes/wheel.dae"/>
       </geometry>
     </collision>
@@ -107,5 +108,5 @@
       <origin xyz="0 0 0" rpy="0 0 0"/>
       <geometry>
-        <mesh filename="file://$(find sec_rob_pkg)/meshes/cover.dae"/>
+        <mesh filename="file://$(find ${pkg_name})/meshes/cover.dae"/>
       </geometry>
       <material name="blue"/>
@@ -114,5 +115,5 @@
       <origin xyz="0 0 0" rpy="0 0 0"/>
       <geometry>
-        <mesh filename="file://$(find sec_rob_pkg)/meshes/cover.dae"/>
+        <mesh filename="file://$(find ${pkg_name})/meshes/cover.dae"/>
       </geometry>
     </collision>
@@ -127,5 +128,5 @@
       <origin xyz="0 0 0" rpy="0 0 0"/>
       <geometry>
-        <mesh filename="file://$(find sec_rob_pkg)/meshes/wheel.dae"/>
+        <mesh filename="file://$(find ${pkg_name})/meshes/wheel.dae"/>
       </geometry>
       <material name="black"/>
@@ -134,5 +135,5 @@
       <origin xyz="0 0 0" rpy="0 0 0"/>
       <geometry>
-        <mesh filename="file://$(find sec_rob_pkg)/meshes/wheel.dae"/>
+        <mesh filename="file://$(find ${pkg_name})/meshes/wheel.dae"/>
       </geometry>
     </collision>
@@ -147,5 +148,5 @@
       <origin xyz="0 0 0" rpy="0 0 0"/>
       <geometry>
-        <mesh filename="file://$(find sec_rob_pkg)/meshes/wheel.dae"/>
+        <mesh filename="file://$(find ${pkg_name})/meshes/wheel.dae"/>
       </geometry>
       <material name="black"/>
@@ -154,5 +155,5 @@
       <origin xyz="0 0 0" rpy="0 0 0"/>
       <geometry>
-        <mesh filename="file://$(find sec_rob_pkg)/meshes/wheel.dae"/>
+        <mesh filename="file://$(find ${pkg_name})/meshes/wheel.dae"/>
       </geometry>
     </collision>
@@ -167,5 +168,5 @@
       <origin xyz="0 0 0" rpy="0 0 0"/>
       <geometry>
-        <mesh filename="file://$(find sec_rob_pkg)/meshes/camera.dae"/>
+        <mesh filename="file://$(find ${pkg_name})/meshes/camera.dae"/>
       </geometry>
       <material name="white"/>
@@ -174,5 +175,5 @@
       <origin xyz="0 0 0" rpy="0 0 0"/>
       <geometry>
-        <mesh filename="file://$(find sec_rob_pkg)/meshes/camera.dae"/>
+        <mesh filename="file://$(find ${pkg_name})/meshes/camera.dae"/>
       </geometry>
     </collision>
@@ -237,3 +238,4 @@
     <child link="camera"/>
   </joint>
+  <xacro:include filename="$(find ${pkg_name})/descriptions/gz_plugins.xacro" />
 </robot>

Commit message: almost there, just ackermann controller not working :{

File: security_robot/src/sr_bringup/descriptions/security_robot.urdf.xacro (robot description, xacro)
@@ -185,5 +185,5 @@
     </inertial>
   </link>
-  <joint name="base_chassis_link" type="fixed">
+  <joint name="base_chassis" type="fixed">
     <parent link="base_link"/>
     <child link="chassis"/>
@@ -238,4 +238,4 @@
     <child link="camera"/>
   </joint>
-  <xacro:include filename="$(find ${pkg_name})/descriptions/gz_plugins.xacro" />
+  <xacro:include filename="$(find ${pkg_name})/descriptions/gz_plugins.gazebo" />
 </robot>
